Commit message: refactor: rename package and update references from ras_robot_simulation to robot_ras_ros

File: urdf/gazebo_elementos.xacro (robot description, xacro)
@@ -6,5 +6,5 @@
                 <plugin>gazebo_ros2_control/GazeboSystem</plugin>
             </hardware>
-            <joint name="esquerda_roda_junta">
+            <joint name="left_wheel_joint">
                 <command_interface name="velocity">
                     <param name="min">-10</param>
@@ -14,5 +14,5 @@
                 <state_interface name="position"/>
             </joint>
-            <joint name="direita_roda_junta">
+            <joint name="right_wheel_joint">
                 <command_interface name="velocity">
                     <param name="min">-10</param>
@@ -26,6 +26,5 @@
             <plugin name="gazebo_ros2_control" filename="libgazebo_ros2_control.so">
                 <robot_param>robot_description</robot_param>
-                <robot_param_node>robot_state_publisher</robot_param_node>
-                <parameters>$(find ras_robot_simulation)/params/ros2_control.yaml</parameters>
+                <parameters>$(find robot_ras_ros)/params/ros2_control.yaml</parameters>
             </plugin>
         </gazebo>

File: urdf/lidar.xacro (robot description, xacro)
@@ -58,6 +58,5 @@
                 <plugin name="${prefix}_range_plugin" filename="libgazebo_ros_ray_sensor.so">
                     <ros>
-                        <namespace>/${prefix}</namespace>
-                        <remapping>~/out:=range</remapping>
+                        <remapping>~/out:=sensor_range/${prefix}</remapping>
                     </ros>
                     <frame_name>${prefix}_lidar_link</frame_name>

File: urdf/robot.urdf.xacro (robot description, xacro)
@@ -10,12 +10,12 @@
     <xacro:include filename="gazebo_elementos.xacro"/>
     <xacro:chassis_macro/>
-    <xacro:roda_macro prefix="esquerda" parent="base_link" y_espelho="-1"/>
-    <xacro:roda_macro prefix="direita" parent="base_link" y_espelho="1"/>
-    <xacro:roda_boba_macro prefix="frente" parent="base_link" x_offset="${pos_x_roda_boba}" y_offset="0" z_offset="${pos_z_roda_boba}"/>
-    <xacro:roda_boba_macro prefix="tras" parent="base_link" x_offset="${-pos_x_roda_boba}" y_offset="0" z_offset="${pos_z_roda_boba}"/>
-    <xacro:lidar_macro prefix="frente" parent="base_link" xyz_origem="${pos_xy_borda_lidar_frente_tras} 0 ${pos_z_lidar}" rpy_origem="0 0 0"/>
-    <xacro:lidar_macro prefix="tras" parent="base_link" xyz_origem="-${pos_xy_borda_lidar_frente_tras} 0 ${pos_z_lidar}" rpy_origem="0 0 ${PI}"/>
-    <xacro:lidar_macro prefix="esquerda" parent="base_link" xyz_origem="0 ${pos_xy_borda_lidar_lados} ${pos_z_lidar}" rpy_origem="0 0 ${PI/2}"/>
-    <xacro:lidar_macro prefix="direita" parent="base_link" xyz_origem="0 -${pos_xy_borda_lidar_lados} ${pos_z_lidar}" rpy_origem="0 0 -${PI/2}"/>
+    <xacro:roda_macro prefix="left" parent="base_link" y_espelho="1"/>
+    <xacro:roda_macro prefix="right" parent="base_link" y_espelho="-1"/>
+    <xacro:roda_boba_macro prefix="front" parent="base_link" x_offset="${pos_x_roda_boba}" y_offset="0" z_offset="${pos_z_roda_boba}"/>
+    <xacro:roda_boba_macro prefix="rear" parent="base_link" x_offset="${-pos_x_roda_boba}" y_offset="0" z_offset="${pos_z_roda_boba}"/>
+    <xacro:lidar_macro prefix="front" parent="base_link" xyz_origem="${pos_xy_borda_lidar_frente_tras} 0 ${pos_z_lidar}" rpy_origem="0 0 0"/>
+    <xacro:lidar_macro prefix="rear" parent="base_link" xyz_origem="-${pos_xy_borda_lidar_frente_tras} 0 ${pos_z_lidar}" rpy_origem="0 0 ${PI}"/>
+    <xacro:lidar_macro prefix="left" parent="base_link" xyz_origem="0.25 ${pos_xy_borda_lidar_lados} ${pos_z_lidar}" rpy_origem="0 0 ${PI/2}"/>
+    <xacro:lidar_macro prefix="right" parent="base_link" xyz_origem="0.25 -${pos_xy_borda_lidar_lados} ${pos_z_lidar}" rpy_origem="0 0 -${PI/2}"/>
     <xacro:gazebo_ros2_control_config/>
 </robot>

File: urdf/roda.xacro (robot description, xacro)
@@ -22,5 +22,5 @@
             </inertial>
         </link>
-        <joint name="${prefix}_roda_junta" type="continuous">
+        <joint name="${prefix}_wheel_joint" type="continuous">
             <parent link="${parent}"/>
             <child link="${prefix}_roda_link"/>
@@ -41,9 +41,7 @@
         <transmission name="${prefix}_roda_transmissao">
             <type>transmission_interface/SimpleTransmission</type>
-            <joint name="${prefix}_roda_junta">
-                <hardwareInterface>hardware_interface/VelocityJointInterface</hardwareInterface>
+            <joint name="${prefix}_wheel_joint">
             </joint>
             <actuator name="${prefix}_roda_motor">
-                <hardwareInterface>hardware_interface/VelocityJointInterface</hardwareInterface>
                 <mechanicalReduction>1</mechanicalReduction>
             </actuator>
