Commit message: feat: add camera and update lidar properties for improved sensor performance

File: urdf/lidar.xacro (robot description, xacro)
@@ -35,5 +35,5 @@
                 <pose>0 0 0 0 0 0</pose>
                 <visualize>true</visualize>
-                <update_rate>20</update_rate>
+                <update_rate>100</update_rate>
                 <ray>
                     <scan>
@@ -46,5 +46,5 @@
                     </scan>
                     <range>
-                        <min>0.10</min>
+                        <min>0.05</min>
                         <max>100.0</max>
                         <resolution>0.01</resolution>
@@ -53,5 +53,5 @@
                         <type>gaussian</type>
                         <mean>0.0</mean>
-                        <stddev>0.02</stddev>
+                        <stddev>0.00</stddev>
                     </noise>
                 </ray>

File: urdf/propriedades.xacro (robot description, xacro)
@@ -2,25 +2,27 @@
 <robot xmlns:xacro="http://www.ros.org/wiki/xacro">
   <xacro:property name="PI" value="3.1415926535897931"/>
-  <xacro:property name="altura_total_robo" value="0.5" />
-  <xacro:property name="largura_total_robo" value="0.9" />
-  <xacro:property name="comprimento_total_robo" value="1.0" />
-  <xacro:property name="comprimento_chassis" value="1.0" />
+  <xacro:property name="fator_escala" value="0.8" />
+  <xacro:property name="fator_escala_cubico" value="${fator_escala * fator_escala * fator_escala}" />
+  <xacro:property name="altura_total_robo" value="${0.5 * fator_escala}" />
+  <xacro:property name="largura_total_robo" value="${0.9 * fator_escala}" />
+  <xacro:property name="comprimento_total_robo" value="${1.0 * fator_escala}" />
+  <xacro:property name="comprimento_chassis" value="${1.0 * fator_escala}" />
   <xacro:property name="largura_chassis" value="${largura_total_robo - 2 * espessura_roda}" />
-  <xacro:property name="altura_chassis" value="0.5" />
-  <xacro:property name="massa_chassis" value="15.0" />
-  <xacro:property name="folga_chao" value="0.1" />
+  <xacro:property name="altura_chassis" value="${0.5 * fator_escala}" />
+  <xacro:property name="massa_chassis" value="${15.0 * fator_escala_cubico}" />
+  <xacro:property name="folga_chao" value="${0.1 * fator_escala}" />
   <xacro:property name="origem_base_link_z_do_chao" value="${folga_chao + altura_chassis/2}" />
-  <xacro:property name="raio_roda" value="0.25" />
-  <xacro:property name="espessura_roda" value="0.05" />
-  <xacro:property name="massa_roda" value="1.0" />
+  <xacro:property name="raio_roda" value="${0.25 * fator_escala}" />
+  <xacro:property name="espessura_roda" value="${0.05 * fator_escala}" />
+  <xacro:property name="massa_roda" value="${1.0 * fator_escala_cubico}" />
   <xacro:property name="pos_x_junta_roda" value="0.0" />
   <xacro:property name="pos_y_junta_roda" value="${largura_chassis/2 + espessura_roda/2}" />
   <xacro:property name="pos_z_junta_roda" value="${raio_roda - origem_base_link_z_do_chao}" />
-  <xacro:property name="raio_roda_boba" value="0.1" />
-  <xacro:property name="massa_roda_boba" value="0.5" />
-  <xacro:property name="pos_x_roda_boba" value="${comprimento_chassis/2 - raio_roda_boba - 0.02}" />
+  <xacro:property name="raio_roda_boba" value="${0.1 * fator_escala}" />
+  <xacro:property name="massa_roda_boba" value="${0.5 * fator_escala_cubico}" />
+  <xacro:property name="pos_x_roda_boba" value="${comprimento_chassis/2 - raio_roda_boba - (0.02 * fator_escala)}" />
   <xacro:property name="pos_z_roda_boba" value="${raio_roda_boba - origem_base_link_z_do_chao}" />
-  <xacro:property name="tamanho_lidar" value="0.05" />
-  <xacro:property name="massa_lidar" value="0.1" />
+  <xacro:property name="tamanho_lidar" value="${0.05 * fator_escala}" />
+  <xacro:property name="massa_lidar" value="${0.1 * fator_escala_cubico}" />
   <xacro:property name="pos_z_lidar" value="${altura_chassis/2 - tamanho_lidar}" />
   <xacro:property name="pos_xy_borda_lidar_frente_tras" value="${comprimento_chassis/2 - tamanho_lidar/4}" />

File: urdf/robot.urdf.xacro (robot description, xacro)
@@ -8,4 +8,5 @@
     <xacro:include filename="roda_boba.xacro"/>
     <xacro:include filename="lidar.xacro"/>
+    <xacro:include filename="camera.xacro"/>
     <xacro:include filename="gazebo_elementos.xacro"/>
     <xacro:chassis_macro/>
@@ -18,4 +19,5 @@
     <xacro:lidar_macro prefix="left" parent="base_link" xyz_origem="0.25 ${pos_xy_borda_lidar_lados} ${pos_z_lidar}" rpy_origem="0 0 ${PI/2}"/>
     <xacro:lidar_macro prefix="right" parent="base_link" xyz_origem="0.25 -${pos_xy_borda_lidar_lados} ${pos_z_lidar}" rpy_origem="0 0 -${PI/2}"/>
+    <xacro:camera_mono_macro prefix="frente" parent="base_link" xyz_origem="${pos_xy_borda_lidar_frente_tras} 0 ${pos_z_lidar - 0.2}" rpy_origem="0 0 0" />
     <xacro:gazebo_ros2_control_config/>
 </robot>
